File: src/メイン回路 Issaimaru側.sch (EAGLE design)
At the start: 4 parts

Commit message: [add]コントローラ
Parts:
- removed JP1, JP2: (no value), pinhead:PINHD-2X19
- removed SV1: (no value), con-ml:ML10L
- removed U$1: A3921, A3921:A3921
- added F303RE_LEFT: (no value), pinhead:PINHD-2X19
- added TWE_L, TWE_R: (no value), pinhead:PINHD-1X14
- added UART: 02-JST, con-jst-xh:02-JST
- added 遠野: (no value), con-ml:ML10
Connections:
- removed net N$1: JP1.15, U$1.GLB
- removed net N$10: JP2.33, SV1.7
- removed net N$11: JP2.31, SV1.9
- removed net N$2: JP1.17, U$1.GHA
- removed net N$3: JP2.10, SV1.1
- removed net N$4: JP2.1, SV1.4
- removed net N$5: JP2.3, SV1.6
- removed net N$6: JP2.5, SV1.8
- removed net N$7: JP2.7, SV1.10
- removed net N$8: JP2.37, SV1.3
- removed net N$9: JP2.35, SV1.5
- new net 3V3: F303RE_LEFT.15, TWE_R.1, 遠野.2
- new net DIR1: F303RE_LEFT.29, 遠野.9
- new net DIR2: F303RE_LEFT.31, 遠野.7
- new net DIR3: F303RE_LEFT.33, 遠野.5
- new net GND: F303RE_LEFT.19, TWE_L.1, 遠野.1
- new net PWM1: F303RE_LEFT.38, 遠野.10
- new net PWM2: F303RE_LEFT.37, 遠野.8
- new net PWM3: F303RE_LEFT.35, 遠野.6
- new net RX_MCU: F303RE_LEFT.1, UART.1
- new net RX_TWE: F303RE_LEFT.18, TWE_L.3
- new net TX_MCU: F303RE_LEFT.2, UART.2
- new net TX_TWE: F303RE_LEFT.16, TWE_L.10
