File: src/コントローラ.brd (EAGLE design)
At the start: 24 parts, among them SW1 TOGGLESWITCH, SW2 TOGGLESWITCH

Commit message: fix
Parts:
- removed JP3, JP4: (no value), con-jst-xh:B3B-XH
- removed R9: (no value), rcl:0207/7
- removed SLIDESWITCH: SLEDESWITCH, slide switch:SLIDESWITCH
- removed SW1, SW2: TOGGLESWITCH, ToggleSwitch:TOGGLESWITCH
- added C1, C2: (no value), rcl:C025-024X044
- added EMAERGENCY: 02-JST, con-jst-xh:B2B-XH
- added JP10, JP11, JP12, JP13, JP14, JP9: (no value), pinhead:1X02
- added JP8, TOGLLESWITCH: (no value), con-jst-xh (1):B3B-XH
- added LED2, LED3, LED4, LED5, LED7: (no value), led:LED5MM
- added R10: 10k, rcl:0204/7
- JP1, JP2: device pinhead:1X05 -> pinhead:1X02
- R7, R8: value (none) -> 10k; device rcl:0207/7 -> rcl:0204/7
- moved R5 305.8 mm to (-2.54, -287.0), turned to 0 degrees
- moved R6 259.2 mm to (-2.54, -298.4)
- moved R8 254.0 mm to (-2.54, -308.6)
- moved R7 254.0 mm to (-2.54, -303.5)
- moved R3 203.3 mm to (-2.54, -222.2)
- moved R4 188.1 mm to (-2.54, -212.1)
- moved JP2 178.9 mm to (-3.81, -113.0)
- moved JP1 156.1 mm to (-3.81, -106.7)
- moved KAHEN 127.0 mm to (-2.54, -171.4)
- moved R1 89.8 mm to (83.8, 6.35), turned to 90 degrees
- moved R2 82.9 mm to (3.81, -39.4), turned to 0 degrees
Connections:
- removed net CONNECT: SLIDESWITCH.1
- removed net CONNECT1: SLIDESWITCH.2
- removed net HORZ1: F303K8_R.9, JP1.3
- removed net HORZ2: F303K8_R.7, JP2.3
- removed net N$2: R8.2, SLIDESWITCH.6
- removed net RT_IN2: BUTTON2.1
- removed net SW_DOWN1: F303K8_L.11, R2.2, SW1.D
- removed net SW_DOWN2: F303K8_L.13, R4.2, SW2.D
- removed net SW_UP1: F303K8_L.10, R1.2, SW1.U
- removed net SW_UP2: F303K8_L.12, R3.2, SW2.U
- removed net SYUUDOUSI＋: R9.2
- removed net VERT1: F303K8_R.10, JP1.2
- removed net VERT2: F303K8_R.8, JP2.2
- removed net VR_IN1: F303K8_R.12, JP3.2
- removed net VR_IN2: F303K8_R.11, JP4.2
- new net AIN5: F303K8_R.6, JP8.2, KAHEN.2, R5.2
- new net L/R1: F303K8_R.10, JP9.2
- new net L/R2: F303K8_R.8, JP11.2
- new net N$3: LED4.A, R8.1
- new net N$4: LED3.A, R7.1
- new net NRST: EMAERGENCY.2, F303K8_R.3
- new net SW\_UP: R3.2, R7.2, TOGLLESWITCH.3
- new net SW_DOWN: F303K8_L.11, R4.2, R6.2, TOGLLESWITCH.1
- new net SW_UP: F303K8_L.10
- new net U/D1: F303K8_R.9, JP1.1
- new net U/D2: F303K8_R.7, JP12.1
- net 3V3: now also C1.1, C2.1, JP11.1, JP8.3, JP9.1, KAHEN.1, TOGLLESWITCH.2; no longer JP1.1, JP2.1, JP3.3, JP4.3, KAHEN.3, SLIDESWITCH.3, SLIDESWITCH.4, SW1.M, SW2.M
- net BT_IN1: now also R1.2, R8.2; no longer R5.2
- net BT_IN2: now also BUTTON2.1, R10.2, R2.2; no longer R6.2
- net GND: now also C1.2, C2.2, EMAERGENCY.1, JP1.2, JP12.2, JP8.1, KAHEN.3, LED2.K, LED3.K, LED4.K, LED5.K, LED7.K; no longer JP1.5, JP2.5, JP3.1, JP4.1, KAHEN.1, R5.1, R6.1, R7.1, R8.1
- net N$1: now also LED7.A, R5.1; no longer R7.2, SLIDESWITCH.5
- net N$5: now also LED2.A, R6.1; no longer KAHEN.2
- net N$7: now also LED5.A, R10.1; no longer R9.1
- net SEL1: no longer JP1.4
- net SEL2: no longer JP2.4
Routing:
- net GND: track 224.3 -> 111.9 mm
- net 3V3: track 204.3 -> 117.9 mm
- net VERT1: track 83.8 -> 0.00 mm
- net HORZ1: track 78.7 -> 0.00 mm
- net VR_IN1: track 73.7 -> 0.00 mm, vias 2 -> 0
- net SW_UP1: track 50.8 -> 0.00 mm, vias 2 -> 0
- net SW_DOWN1: track 45.7 -> 0.00 mm, vias 2 -> 0
- net VR_IN2: track 45.3 -> 0.00 mm
- net HORZ2: track 38.1 -> 0.00 mm
- net SW_UP: track 0.00 -> 35.6 mm, vias 0 -> 2
- net SW_DOWN: track 0.00 -> 35.6 mm, vias 0 -> 2
- net VERT2: track 33.0 -> 0.00 mm
- net SEL2: track 78.7 -> 58.4 mm
- net SEL1: track 35.6 -> 30.5 mm

Commit message: [add]コントローラAoi
Parts:
- removed LED7: (no value), led:LED5MM
- removed R10: 10k, rcl:0204/7
- added LED1, LED6: 02-JST, con-jst-xh (1):B2B-XH
- added R11, R9: 100, rcl:0204/7
- LED2, LED3, LED4, LED5: value (none) -> 02-JST; device led:LED5MM -> con-jst-xh (1):B2B-XH
- R5, R6, R7, R8: value 10k -> 100
- moved LED5 317.4 mm to (64.8, 36.8), turned to 270 degrees
- moved LED4 308.6 mm to (58.4, 36.8), turned to 270 degrees
- moved EMAERGENCY 307.3 mm to (87.6, 58.4)
- moved LED2 302.9 mm to (15.2, 52.1), turned to 270 degrees
- moved LED3 300.3 mm to (15.2, 41.9), turned to 270 degrees
- moved R5 287.2 mm to (-57.1, -5.08)
- moved R3 270.2 mm to (20.3, 47.0), turned to 270 degrees
- moved R6 268.5 mm to (-57.1, -35.6)
- moved TOGLLESWITCH 260.9 mm to (27.9, 53.3), turned to 270 degrees
- moved R7 258.6 mm to (-57.1, -50.8)
- moved R8 248.6 mm to (-57.1, -66.0)
- moved R4 243.9 mm to (82.5, 16.5), turned to 90 degrees
- moved KAHEN 229.5 mm to (78.7, 43.2), turned to 90 degrees
- moved C2 221.6 mm to (88.9, 34.3), turned to 270 degrees
- moved JP13 211.9 mm to (88.9, 29.2), turned to 90 degrees
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Connections:
- removed net N$3: LED4.A, R8.1
- removed net N$4: LED3.A, R7.1
- removed net N$5: LED2.A, R6.1
- removed net N$7: LED5.A, R10.1
- new net D1: F303K8_L.12, LED1.2, R5.1, TWE_R.14
- net AIN5: now also LED6.2, R9.1; no longer R5.2
- net BT_IN1: now also LED2.2, R11.1; no longer R8.2
- net BT_IN2: now also LED3.2, R6.1; no longer R10.2
- net GND: now also LED1.1, LED2.1, LED3.1, LED4.1, LED5.1, LED6.1, R11.2, R5.2, R6.2, R7.2, R8.2, R9.2; no longer C1.2, JP1.2, LED2.K, LED3.K, LED4.K, LED5.K, LED7.K
- net N$1: now also C1.2, JP1.2; no longer LED7.A, R5.1
- net SW\_UP: no longer R7.2
- net SW_DOWN: now also LED5.2, R8.1; no longer R6.2
- net SW_UP: now also LED4.2, R7.1
Routing:
- net GND: track 111.9 -> 219.7 mm, vias 0 -> 4
- net L/R1: track 0.00 -> 75.2 mm
- net AIN5: track 0.00 -> 73.7 mm, vias 0 -> 2
- net U/D2: track 0.00 -> 63.5 mm
- net BT_IN1: track 119.4 -> 59.7 mm, vias 2 -> 0
- net SEL2: track 58.4 -> 0.00 mm, vias 2 -> 0
- net D1: track 0.00 -> 50.8 mm
- net BT_IN2: track 0.00 -> 48.3 mm
- net N$1: track 0.00 -> 45.7 mm
- net 3V3: track 117.9 -> 157.5 mm, vias 2 -> 4
- net L/R2: track 0.00 -> 35.6 mm, vias 0 -> 2
- net NRST: track 0.00 -> 33.0 mm
- net SEL1: track 30.5 -> 0.00 mm
- net SW_DOWN: track 35.6 -> 12.7 mm
- net SW_UP: track 35.6 -> 20.3 mm, vias 2 -> 1
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
Commit message: [add]コントローラ　Aoi
Parts:
- removed R11: 100, rcl:0204/7
- removed TOGLLESWITCH: (no value), con-jst-xh (1):B3B-XH
- added PIN, PINSOCKET: (no value), pinhead:1X15
- added R10: 100, rcl:0204/7
- added TOGGLESWITCH: (no value), con-jst-xh (1):B3B-XH
- added U$2: (no value), prototyping-board (2):TYPE.C
- moved R9 187.6 mm to (19.1, 90.2)
- moved R8 172.7 mm to (21.6, 87.6)
- moved R7 169.4 mm to (36.8, 90.2)
- moved R6 156.5 mm to (39.4, 87.6)
- moved LED5 87.7 mm to (15.2, 109.2)
- moved R4 79.3 mm to (17.8, 62.2), turned to 270 degrees
- moved LED4 77.8 mm to (15.2, 101.6)
- moved R5 76.7 mm to (10.2, 31.8), turned to 90 degrees
- moved LED3 71.9 mm to (40.6, 109.2)
- moved BUTTON2 71.2 mm to (26.7, 110.5), turned to 0 degrees
- moved LED2 55.7 mm to (40.6, 101.6)
- moved BUTTON 54.3 mm to (26.7, 102.9), turned to 0 degrees
- moved JP8 43.5 mm to (71.1, 68.6)
- moved LED6 37.2 mm to (58.4, 104.1)
- moved R3 17.8 mm to (20.3, 64.8)
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Connections:
- removed net SW\_UP: R3.2, TOGLLESWITCH.3
- new net N$8: PINSOCKET.3
- net 3V3: now also PIN.15, PINSOCKET.15, TOGGLESWITCH.2; no longer TOGLLESWITCH.2
- net AIN5: now also PIN.14, PINSOCKET.14, R10.1; no longer R9.1
- net BT_IN1: now also PIN.7, PINSOCKET.7, R6.1; no longer R11.1
- net BT_IN2: now also F303K8_L.10, PIN.6, PINSOCKET.6, R7.1; no longer F303K8_L.14, R6.1
- net D1: now also F303K8_L.14; no longer F303K8_L.12
- net GND: now also C1.2, JP1.2, PIN.13, PINSOCKET.13, R10.2; no longer R11.2
- net N$1: now also PIN.3; no longer C1.2, JP1.2
- net SW_DOWN: now also F303K8_L.12, PIN.4, PINSOCKET.4, R9.1, TOGGLESWITCH.3; no longer F303K8_L.11, R8.1, TOGLLESWITCH.1
- net SW_UP: now also F303K8_L.11, PIN.5, PINSOCKET.5, R3.2, R8.1, TOGGLESWITCH.1; no longer F303K8_L.10, R7.1
Routing:
- net GND: track 219.7 -> 494.4 mm, vias 4 -> 6
- net 3V3: track 157.5 -> 356.9 mm
- net U/D1: track 8.89 -> 114.3 mm, vias 0 -> 6
- net SW_DOWN: track 12.7 -> 116.8 mm, vias 2 -> 0
- net SW_UP: track 20.3 -> 114.3 mm, vias 1 -> 2
- net N$1: track 45.7 -> 0.00 mm
- net AIN5: track 73.7 -> 111.8 mm
- net BT_IN2: track 48.3 -> 86.4 mm, vias 0 -> 2
- net L/R1: track 75.2 -> 106.7 mm, vias 0 -> 4
- net BT_IN1: track 59.7 -> 73.7 mm
- net D1: track 50.8 -> 63.5 mm, vias 0 -> 2
- net NRST: track 33.0 -> 43.2 mm
- net U/D2: track 63.5 -> 73.7 mm
- net TX: track 44.5 -> 39.4 mm
- net SW\_UP: track 5.08 -> 0.00 mm, vias 1 -> 0
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
Commit message: [add]コントローラ　Aoi
Parts:
- moved C1 15.2 mm to (22.9, 52.1)
- moved C2 15.2 mm to (88.9, 52.1)
- moved JP11 15.2 mm to (71.1, 47.0)
- moved JP13 15.2 mm to (88.9, 47.0)
- moved JP2 15.2 mm to (22.9, 47.0)
- moved JP9 15.2 mm to (5.08, 47.0)
- moved JP1 15.2 mm to (5.08, 24.1)
- moved JP10 15.2 mm to (22.9, 24.1)
- moved JP12 15.2 mm to (71.1, 24.1)
- moved JP14 15.2 mm to (88.9, 24.1)
- moved KAHEN 11.4 mm to (83.8, 55.9)
Routing:
- net AIN5: track 111.8 -> 84.9 mm
- net U/D1: track 114.3 -> 128.1 mm
- net L/R1: track 106.7 -> 113.9 mm
- net U/D2: track 73.7 -> 67.1 mm
- net RX: track 34.3 -> 40.6 mm
- net TX: track 39.4 -> 43.2 mm
- net GND: track 494.4 -> 498.0 mm
- net 3V3: track 356.9 -> 353.9 mm
- net L/R2: track 40.6 -> 39.2 mm, vias 2 -> 0
- net N$2: track 1.27 -> 0.00 mm
