File: src/2022国技館射出.sch (EAGLE design)
At the start: 29 parts

Commit message: 国技館足回り回路の追加
Parts:
- removed UART: 02-JST, con-jst-xh:02-JST
- added MAT_LED, SUSPENSION: 02-JST, con-jst-xh:02-JST
Connections:
- removed net RX: JP5.4, UART.1
- removed net TX: JP5.3, UART.2
- new net RX1: JP5.4, SUSPENSION.1
- new net RX2: JP5.9, MAT_LED.1
- new net TX1: JP5.3, SUSPENSION.2
- new net TX2: JP5.11, MAT_LED.2
Changed lines of the file:
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@@
 <part name="SV2" library="con-ml" library_urn="urn:adsk.eagle:library:164" deviceset="ML10" device="" package3d_urn="urn:adsk.eagle:package:8676/1"/>
 <part name="POW" library="con-jst-xh" deviceset="02-JST" device=""/>
-<part name="UART" library="con-jst-xh" deviceset="02-JST" device=""/>
+<part name="SUSPENSION" library="con-jst-xh" deviceset="02-JST" device=""/>
 <part name="C1" library="rcl" library_urn="urn:adsk.eagle:library:334" deviceset="C-EU" device="025-024X044" package3d_urn="urn:adsk.eagle:package:23630/1"/>
 <part name="JP9" library="con-jst-xh" deviceset="04-JST" device=""/>
@@
 <part name="R6" library="rcl" library_urn="urn:adsk.eagle:library:334" deviceset="R-EU_" device="0204/7" package3d_urn="urn:adsk.eagle:package:23498/2" value="100"/>
 <part name="R7" library="rcl" library_urn="urn:adsk.eagle:library:334" deviceset="R-EU_" device="0204/7" package3d_urn="urn:adsk.eagle:package:23498/2" value="100"/>
+<part name="MAT_LED" library="con-jst-xh" deviceset="02-JST" device=""/>
 </parts>
 <sheets>
@@
 <wire x1="81.28" y1="71.12" x2="40.64" y2="71.12" width="0.1524" layer="97"/>
 <text x="55.88" y="40.64" size="1.778" layer="97">POW</text>
-<wire x1="30.48" y1="213.36" x2="30.48" y2="185.42" width="0.1524" layer="97"/>
+<wire x1="30.48" y1="226.06" x2="30.48" y2="185.42" width="0.1524" layer="97"/>
 <wire x1="30.48" y1="185.42" x2="66.04" y2="185.42" width="0.1524" layer="97"/>
-<wire x1="66.04" y1="185.42" x2="66.04" y2="213.36" width="0.1524" layer="97"/>
-<wire x1="66.04" y1="213.36" x2="30.48" y2="213.36" width="0.1524" layer="97"/>
+<wire x1="66.04" y1="185.42" x2="66.04" y2="226.06" width="0.1524" layer="97"/>
+<wire x1="66.04" y1="226.06" x2="30.48" y2="226.06" width="0.1524" layer="97"/>
 <text x="45.72" y="182.88" size="1.778" layer="97">UART</text>
 <wire x1="284.48" y1="137.16" x2="284.48" y2="111.76" width="0.1524" layer="97"/>
@@
 <attribute name="NAME" x="49.53" y="61.722" size="1.778" layer="95"/>
 </instance>
-<instance part="UART" gate="G$1" x="43.18" y="200.66" smashed="yes">
-<attribute name="VALUE" x="41.91" y="193.04" size="1.778" layer="96"/>
-<attribute name="NAME" x="41.91" y="203.962" size="1.778" layer="95"/>
+<instance part="SUSPENSION" gate="G$1" x="43.18" y="213.36" smashed="yes">
+<attribute name="VALUE" x="41.91" y="205.74" size="1.778" layer="96"/>
+<attribute name="NAME" x="41.91" y="216.662" size="1.778" layer="95"/>
 </instance>
 <instance part="C1" gate="G$1" x="63.5" y="58.42" smashed="yes">
@@
 <attribute name="NAME" x="306.07" y="98.0186" size="1.778" layer="95"/>
 <attribute name="VALUE" x="307.848" y="95.758" size="1.778" layer="96"/>
+</instance>
+<instance part="MAT_LED" gate="G$1" x="43.18" y="198.12" smashed="yes">
+<attribute name="VALUE" x="41.91" y="190.5" size="1.778" layer="96"/>
+<attribute name="NAME" x="41.91" y="201.422" size="1.778" layer="95"/>
 </instance>
 </instances>
@@
 </segment>
 </net>
-<net name="TX" class="0">
-<segment>
-<pinref part="JP5" gate="A" pin="3"/>
-<wire x1="154.94" y1="193.04" x2="139.7" y2="193.04" width="0.1524" layer="91"/>
-<label x="139.7" y="193.04" size="1.778" layer="95"/>
-</segment>
-<segment>
-<pinref part="UART" gate="G$1" pin="2"/>
-<wire x1="50.8" y1="200.66" x2="58.42" y2="200.66" width="0.1524" layer="91"/>
-<label x="55.88" y="200.66" size="1.778" layer="95"/>
-</segment>
-</net>
-<net name="RX" class="0">
-<segment>
-<pinref part="JP5" gate="A" pin="4"/>
-<wire x1="162.56" y1="193.04" x2="172.72" y2="193.04" width="0.1524" layer="91"/>
-<label x="170.18" y="193.04" size="1.778" layer="95"/>
-</segment>
-<segment>
-<pinref part="UART" gate="G$1" pin="1"/>
-<wire x1="50.8" y1="198.12" x2="58.42" y2="198.12" width="0.1524" layer="91"/>
-<label x="55.88" y="198.12" size="1.778" layer="95"/>
-</segment>
-</net>
 <net name="BLUE" class="0">
 <segment>
@@
 </segment>
 </net>
+<net name="TX1" class="0">
+<segment>
+<pinref part="JP5" gate="A" pin="3"/>
+<wire x1="154.94" y1="193.04" x2="139.7" y2="193.04" width="0.1524" layer="91"/>
+<label x="139.7" y="193.04" size="1.778" layer="95"/>
+</segment>
+<segment>
+<pinref part="SUSPENSION" gate="G$1" pin="2"/>
+<wire x1="50.8" y1="213.36" x2="58.42" y2="213.36" width="0.1524" layer="91"/>
+<label x="55.88" y="213.36" size="1.778" layer="95"/>
+</segment>
+</net>
+<net name="RX1" class="0">
+<segment>
+<pinref part="JP5" gate="A" pin="4"/>
+<wire x1="162.56" y1="193.04" x2="172.72" y2="193.04" width="0.1524" layer="91"/>
+<label x="170.18" y="193.04" size="1.778" layer="95"/>
+</segment>
+<segment>
+<pinref part="SUSPENSION" gate="G$1" pin="1"/>
+<wire x1="50.8" y1="210.82" x2="58.42" y2="210.82" width="0.1524" layer="91"/>
+<label x="55.88" y="210.82" size="1.778" layer="95"/>
+</segment>
+</net>
+<net name="RX2" class="0">
+<segment>
+<pinref part="JP5" gate="A" pin="9"/>
+<wire x1="154.94" y1="185.42" x2="139.7" y2="185.42" width="0.1524" layer="91"/>
+<label x="139.7" y="185.42" size="1.778" layer="95"/>
+</segment>
+<segment>
+<pinref part="MAT_LED" gate="G$1" pin="1"/>
+<wire x1="50.8" y1="195.58" x2="58.42" y2="195.58" width="0.1524" layer="91"/>
+<label x="55.88" y="195.58" size="1.778" layer="95"/>
+</segment>
+</net>
+<net name="TX2" class="0">
+<segment>
+<pinref part="JP5" gate="A" pin="11"/>
+<wire x1="154.94" y1="182.88" x2="139.7" y2="182.88" width="0.1524" layer="91"/>
+<label x="139.7" y="182.88" size="1.778" layer="95"/>
+</segment>
+<segment>
+<pinref part="MAT_LED" gate="G$1" pin="2"/>
+<wire x1="50.8" y1="198.12" x2="58.42" y2="198.12" width="0.1524" layer="91"/>
+<label x="55.88" y="198.12" size="1.778" layer="95"/>
+</segment>
+</net>

Commit message: 2022/11/03
Connections:
- net GND: no longer JP5.49
- net PWM1: now also JP6.33; no longer JP6.27
- net PWM2: now also JP6.31; no longer JP6.29
- net PWM3: now also JP6.29; no longer JP6.31
- net PWM4: now also JP6.27; no longer JP6.33
- net PWM5: now also JP6.37; no longer JP6.35
- net PWM6: now also JP6.35; no longer JP6.37
Changed lines of the file:
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@@
-</segment>
-<segment>
-<pinref part="JP5" gate="A" pin="49"/>
-<wire x1="154.94" y1="134.62" x2="139.7" y2="134.62" width="0.1524" layer="91"/>
-<label x="139.7" y="134.62" size="1.778" layer="95"/>
 </segment>
 <segment>
@@
 <net name="PWM6" class="0">
 <segment>
-<pinref part="JP6" gate="A" pin="37"/>
-<wire x1="203.2" y1="149.86" x2="190.5" y2="149.86" width="0.1524" layer="91"/>
-<label x="190.5" y="149.86" size="1.778" layer="95"/>
-</segment>
-<segment>
 <pinref part="SV2" gate="G$1" pin="8"/>
 <wire x1="304.8" y1="167.64" x2="297.18" y2="167.64" width="0.1524" layer="91"/>
 <label x="297.18" y="167.64" size="1.778" layer="95"/>
 </segment>
-</net>
-<net name="PWM5" class="0">
 <segment>
 <pinref part="JP6" gate="A" pin="35"/>
@@
 <label x="190.5" y="152.4" size="1.778" layer="95"/>
 </segment>
+</net>
+<net name="PWM5" class="0">
 <segment>
 <pinref part="SV2" gate="G$1" pin="10"/>
@@
 <label x="297.18" y="170.18" size="1.778" layer="95"/>
 </segment>
+<segment>
+<pinref part="JP6" gate="A" pin="37"/>
+<wire x1="203.2" y1="149.86" x2="190.5" y2="149.86" width="0.1524" layer="91"/>
+<label x="190.5" y="149.86" size="1.778" layer="95"/>
+</segment>
 </net>
 <net name="PWM4" class="0">
+<segment>
+<pinref part="SV1" gate="G$1" pin="4"/>
+<wire x1="304.8" y1="187.96" x2="297.18" y2="187.96" width="0.1524" layer="91"/>
+<label x="297.18" y="187.96" size="1.778" layer="95"/>
+</segment>
+<segment>
+<pinref part="JP6" gate="A" pin="27"/>
+<wire x1="203.2" y1="162.56" x2="190.5" y2="162.56" width="0.1524" layer="91"/>
+<label x="190.5" y="162.56" size="1.778" layer="95"/>
+</segment>
+</net>
+<net name="PWM3" class="0">
+<segment>
+<pinref part="SV1" gate="G$1" pin="6"/>
+<wire x1="304.8" y1="190.5" x2="297.18" y2="190.5" width="0.1524" layer="91"/>
+<label x="297.18" y="190.5" size="1.778" layer="95"/>
+</segment>
+<segment>
+<pinref part="JP6" gate="A" pin="29"/>
+<wire x1="203.2" y1="160.02" x2="190.5" y2="160.02" width="0.1524" layer="91"/>
+<label x="190.5" y="160.02" size="1.778" layer="95"/>
+</segment>
+</net>
+<net name="PWM2" class="0">
+<segment>
+<pinref part="SV1" gate="G$1" pin="8"/>
+<wire x1="304.8" y1="193.04" x2="297.18" y2="193.04" width="0.1524" layer="91"/>
+<label x="297.18" y="193.04" size="1.778" layer="95"/>
+</segment>
+<segment>
+<pinref part="JP6" gate="A" pin="31"/>
+<wire x1="203.2" y1="157.48" x2="190.5" y2="157.48" width="0.1524" layer="91"/>
+<label x="190.5" y="157.48" size="1.778" layer="95"/>
+</segment>
+</net>
+<net name="PWM1" class="0">
+<segment>
+<pinref part="SV1" gate="G$1" pin="10"/>
+<wire x1="304.8" y1="195.58" x2="297.18" y2="195.58" width="0.1524" layer="91"/>
+<label x="297.18" y="195.58" size="1.778" layer="95"/>
+</segment>
 <segment>
 <pinref part="JP6" gate="A" pin="33"/>
@@
 <label x="190.5" y="154.94" size="1.778" layer="95"/>
 </segment>
-<segment>
-<pinref part="SV1" gate="G$1" pin="4"/>
-<wire x1="304.8" y1="187.96" x2="297.18" y2="187.96" width="0.1524" layer="91"/>
-<label x="297.18" y="187.96" size="1.778" layer="95"/>
-</segment>
 </net>
-<net name="PWM3" class="0">
-<segment>
-<pinref part="JP6" gate="A" pin="31"/>
-<wire x1="203.2" y1="157.48" x2="190.5" y2="157.48" width="0.1524" layer="91"/>
-<label x="190.5" y="157.48" size="1.778" layer="95"/>
-</segment>
-<segment>
-<pinref part="SV1" gate="G$1" pin="6"/>
-<wire x1="304.8" y1="190.5" x2="297.18" y2="190.5" width="0.1524" layer="91"/>
-<label x="297.18" y="190.5" size="1.778" layer="95"/>
-</segment>
-</net>
-<net name="PWM2" class="0">
-<segment>
-<pinref part="JP6" gate="A" pin="29"/>
-<wire x1="203.2" y1="160.02" x2="190.5" y2="160.02" width="0.1524" layer="91"/>
-<label x="190.5" y="160.02" size="1.778" layer="95"/>
-</segment>
-<segment>
-<pinref part="SV1" gate="G$1" pin="8"/>
-<wire x1="304.8" y1="193.04" x2="297.18" y2="193.04" width="0.1524" layer="91"/>
-<label x="297.18" y="193.04" size="1.778" layer="95"/>
-</segment>
-</net>
-<net name="PWM1" class="0">
-<segment>
-<pinref part="JP6" gate="A" pin="27"/>
-<wire x1="203.2" y1="162.56" x2="190.5" y2="162.56" width="0.1524" layer="91"/>
-<label x="190.5" y="162.56" size="1.778" layer="95"/>
-</segment>
-<segment>
-<pinref part="SV1" gate="G$1" pin="10"/>
-<wire x1="304.8" y1="195.58" x2="297.18" y2="195.58" width="0.1524" layer="91"/>
-<label x="297.18" y="195.58" size="1.778" layer="95"/>
-</segment>
-</net>

Commit message: 2022国技館射出完成
Connections:
- net DIR1: now also JP6.19; no longer JP6.25
- net DIR2: now also JP6.21; no longer JP6.23
- net DIR3: now also JP6.23; no longer JP6.21
- net DIR4: now also JP6.25; no longer JP6.19
- net DIR5: now also JP6.15; no longer JP6.17
- net DIR6: now also JP6.17; no longer JP6.15
- net GND: now also JP6.54
Changed lines of the file:
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@@
 <junction x="330.2" y="83.82"/>
+</segment>
+<segment>
+<pinref part="JP6" gate="A" pin="54"/>
+<wire x1="210.82" y1="129.54" x2="223.52" y2="129.54" width="0.1524" layer="91"/>
+<label x="218.44" y="129.54" size="1.778" layer="95"/>
 </segment>
 </net>
@@
 <net name="DIR1" class="0">
 <segment>
-<pinref part="JP6" gate="A" pin="25"/>
-<wire x1="203.2" y1="165.1" x2="190.5" y2="165.1" width="0.1524" layer="91"/>
-<label x="190.5" y="165.1" size="1.778" layer="95"/>
-</segment>
-<segment>
 <pinref part="SV1" gate="G$1" pin="9"/>
 <wire x1="320.04" y1="195.58" x2="327.66" y2="195.58" width="0.1524" layer="91"/>
 <label x="322.58" y="195.58" size="1.778" layer="95"/>
 </segment>
+<segment>
+<pinref part="JP6" gate="A" pin="19"/>
+<wire x1="203.2" y1="172.72" x2="190.5" y2="172.72" width="0.1524" layer="91"/>
+<label x="190.5" y="172.72" size="1.778" layer="95"/>
+</segment>
 </net>
 <net name="DIR2" class="0">
+<segment>
+<pinref part="SV1" gate="G$1" pin="7"/>
+<wire x1="320.04" y1="193.04" x2="327.66" y2="193.04" width="0.1524" layer="91"/>
+<label x="322.58" y="193.04" size="1.778" layer="95"/>
+</segment>
+<segment>
+<pinref part="JP6" gate="A" pin="21"/>
+<wire x1="203.2" y1="170.18" x2="190.5" y2="170.18" width="0.1524" layer="91"/>
+<label x="190.5" y="170.18" size="1.778" layer="95"/>
+</segment>
+</net>
+<net name="DIR3" class="0">
+<segment>
+<pinref part="SV1" gate="G$1" pin="5"/>
+<wire x1="320.04" y1="190.5" x2="327.66" y2="190.5" width="0.1524" layer="91"/>
+<label x="322.58" y="190.5" size="1.778" layer="95"/>
+</segment>
 <segment>
 <pinref part="JP6" gate="A" pin="23"/>
@@
 <label x="190.5" y="167.64" size="1.778" layer="95"/>
 </segment>
+</net>
+<net name="DIR5" class="0">
 <segment>
-<pinref part="SV1" gate="G$1" pin="7"/>
-<wire x1="320.04" y1="193.04" x2="327.66" y2="193.04" width="0.1524" layer="91"/>
-<label x="322.58" y="193.04" size="1.778" layer="95"/>
+<pinref part="SV2" gate="G$1" pin="9"/>
+<wire x1="320.04" y1="170.18" x2="327.66" y2="170.18" width="0.1524" layer="91"/>
+<label x="322.58" y="170.18" size="1.778" layer="95"/>
+</segment>
+<segment>
+<pinref part="JP6" gate="A" pin="15"/>
+<wire x1="203.2" y1="177.8" x2="190.5" y2="177.8" width="0.1524" layer="91"/>
+<label x="190.5" y="177.8" size="1.778" layer="95"/>
 </segment>
 </net>
-<net name="DIR3" class="0">
+<net name="DIR6" class="0">
 <segment>
-<pinref part="JP6" gate="A" pin="21"/>
-<wire x1="203.2" y1="170.18" x2="190.5" y2="170.18" width="0.1524" layer="91"/>
-<label x="190.5" y="170.18" size="1.778" layer="95"/>
+<pinref part="SV2" gate="G$1" pin="7"/>
+<wire x1="320.04" y1="167.64" x2="327.66" y2="167.64" width="0.1524" layer="91"/>
+<label x="322.58" y="167.64" size="1.778" layer="95"/>
 </segment>
-<segment>
-<pinref part="SV1" gate="G$1" pin="5"/>
-<wire x1="320.04" y1="190.5" x2="327.66" y2="190.5" width="0.1524" layer="91"/>
-<label x="322.58" y="190.5" size="1.778" layer="95"/>
-</segment>
-</net>
-<net name="DIR5" class="0">
 <segment>
 <pinref part="JP6" gate="A" pin="17"/>
@@
 <label x="190.5" y="175.26" size="1.778" layer="95"/>
 </segment>
-<segment>
-<pinref part="SV2" gate="G$1" pin="9"/>
-<wire x1="320.04" y1="170.18" x2="327.66" y2="170.18" width="0.1524" layer="91"/>
-<label x="322.58" y="170.18" size="1.778" layer="95"/>
-</segment>
-</net>
-<net name="DIR6" class="0">
-<segment>
-<pinref part="JP6" gate="A" pin="15"/>
-<wire x1="203.2" y1="177.8" x2="190.5" y2="177.8" width="0.1524" layer="91"/>
-<label x="190.5" y="177.8" size="1.778" layer="95"/>
-</segment>
-<segment>
-<pinref part="SV2" gate="G$1" pin="7"/>
-<wire x1="320.04" y1="167.64" x2="327.66" y2="167.64" width="0.1524" layer="91"/>
-<label x="322.58" y="167.64" size="1.778" layer="95"/>
-</segment>
 </net>
 <net name="DIR4" class="0">
-<segment>
-<pinref part="JP6" gate="A" pin="19"/>
-<wire x1="203.2" y1="172.72" x2="190.5" y2="172.72" width="0.1524" layer="91"/>
-<label x="190.5" y="172.72" size="1.778" layer="95"/>
-</segment>
 <segment>
 <pinref part="SV1" gate="G$1" pin="3"/>
@@
 <label x="322.58" y="187.96" size="1.778" layer="95"/>
 </segment>
+<segment>
+<pinref part="JP6" gate="A" pin="25"/>
+<wire x1="203.2" y1="165.1" x2="190.5" y2="165.1" width="0.1524" layer="91"/>
+<label x="190.5" y="165.1" size="1.778" layer="95"/>
+</segment>
 </net>
