File: src/2022国技館射出.brd (EAGLE design)
At the start: 31 parts

Commit message: 国技館足回り回路の追加
Parts:
- added MAT_LED: 02-JST, con-jst-xh:B2B-XH
- moved SV1 332.9 mm to (194.3, 128.3), turned to 270 degrees
- moved SV2 323.1 mm to (194.3, 97.8), turned to 270 degrees
- renumbered UART to SUSPENSION
Connections:
- net RX renamed RX1
- net TX renamed TX1
- new net RX2: JP5.9, MAT_LED.1
- new net TX2: JP5.11, MAT_LED.2

Commit message: 2022/11/03
Parts:
- moved LED6 365.5 mm to (207.0, 54.6)
- moved R6 349.3 mm to (168.9, 52.1)
- moved LED4 349.1 mm to (196.8, 54.6)
- moved LED5 347.9 mm to (196.8, 44.5)
- moved R5 347.8 mm to (168.9, 54.6)
- moved R4 346.2 mm to (168.9, 57.1)
- moved R3 344.7 mm to (168.9, 59.7)
- moved MAT_LED 343.7 mm to (54.6, 133.3)
- moved R2 343.2 mm to (168.9, 62.2)
- moved JP9 337.4 mm to (193.0, 71.1), turned to 270 degrees
- moved LED2 332.9 mm to (186.7, 54.6)
- moved LED3 331.7 mm to (186.7, 44.5)
- moved SUSPENSION 272.3 mm to (54.6, 143.5)
- moved R7 253.8 mm to (47.0, 34.3), turned to 180 degrees
- moved R1 228.4 mm to (47.0, 31.8), turned to 180 degrees
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Connections:
- net GND: no longer JP5.49
- net PWM1: now also JP6.33; no longer JP6.27
- net PWM2: now also JP6.31; no longer JP6.29
- net PWM3: now also JP6.29; no longer JP6.31
- net PWM4: now also JP6.27; no longer JP6.33
- net PWM5: now also JP6.37; no longer JP6.35
- net PWM6: now also JP6.35; no longer JP6.37
Routing:
- net GND: track 0.00 -> 401.3 mm, vias 0 -> 10
- net 5V: track 0.00 -> 271.8 mm
- net VIN: track 0.00 -> 134.6 mm
- net 3V3: track 0.00 -> 124.5 mm
- net PWM4: track 0.00 -> 96.5 mm
- net PWM6: track 0.00 -> 94.0 mm
- net PWM3: track 0.00 -> 91.4 mm
- net PWM5: track 0.00 -> 88.9 mm
- net PWM2: track 0.00 -> 86.4 mm
- net ENC1_A: track 0.00 -> 83.8 mm
- net PWM1: track 0.00 -> 81.3 mm
- net ENC2_A: track 0.00 -> 78.7 mm
- net ENC3_A: track 0.00 -> 76.2 mm
- net ENC1_B: track 0.00 -> 76.2 mm
- net N$6: track 0.00 -> 71.1 mm
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
Commit message: 2022国技館射出完成
Parts:
- moved JP9 5.08 mm to (193.0, 76.2)
- moved SV2 3.59 mm to (170.2, 25.4)
- moved SV1 3.59 mm to (147.3, 25.4)
Connections:
- net DIR1: now also JP6.19; no longer JP6.25
- net DIR2: now also JP6.21; no longer JP6.23
- net DIR3: now also JP6.23; no longer JP6.21
- net DIR4: now also JP6.25; no longer JP6.19
- net DIR5: now also JP6.15; no longer JP6.17
- net DIR6: now also JP6.17; no longer JP6.15
- net GND: now also JP6.54
Routing:
- net DIR6: track 0.00 -> 271.8 mm
- net DIR5: track 0.00 -> 246.4 mm
- net DIR1: track 0.00 -> 167.6 mm
- net DIR2: track 0.00 -> 152.4 mm
- net GND: track 401.3 -> 551.2 mm, vias 10 -> 14
- net 3V3: track 124.5 -> 266.7 mm, vias 0 -> 4
- net DIR3: track 0.00 -> 137.2 mm
- net DIR4: track 0.00 -> 121.9 mm
- net BLUE: track 38.1 -> 33.0 mm
- net RED: track 40.6 -> 35.6 mm
- net GREEN: track 40.6 -> 35.6 mm

Commit message: 11/08修正
Parts:
- moved C1 10.2 mm to (96.5, 111.8)
- moved JP5 10.2 mm to (90.2, 100.3)
- moved JP7 10.2 mm to (90.2, 55.9)
Routing:
- net GND: track 551.2 -> 561.3 mm
- net VIN: track 134.6 -> 144.8 mm
- net RX1: track 38.1 -> 48.3 mm
- net ENC3_B: track 68.6 -> 78.7 mm
- net ENC1_B: track 76.2 -> 86.4 mm
- net ENC5_B: track 58.4 -> 68.6 mm
- net TX2: track 33.0 -> 43.2 mm
- net TX1: track 33.0 -> 43.2 mm
- net RX2: track 27.9 -> 38.1 mm
- net ENC6_B: track 53.3 -> 63.5 mm
- net ENC5_A: track 66.0 -> 76.2 mm
- net ENC4_A: track 71.1 -> 81.3 mm
- net ENC3_A: track 76.2 -> 86.4 mm
- net ENC2_A: track 78.7 -> 88.9 mm
- net ENC6_A: track 61.0 -> 71.1 mm
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